File: pcb/cantorplus.kicad_pcb (KiCad board)
At the start: 2 copper layers, 138.8 x 91.8 mm, 23 parts, among them J1 TRRS, K00 KEYSW, K01 KEYSW, K02 KEYSW, K03 KEYSW, K04 KEYSW, K05 KEYSW, K10 KEYSW, K11 KEYSW, K12 KEYSW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

Commit message: Updated kicad files
Other:
- board text added: "U1"
Changed lines of the file:
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@@
     (property "Sheetname" "")
     (attr through_hole)
-    (fp_text reference "K32" (at 0 -8.255 155) (layer "F.SilkS")
+    (fp_text reference "K32" (at 0 -8.255 -25 unlocked) (layer "F.SilkS")
       (effects (font (size 1 1) (thickness 0.15)))
     )
@@
       (effects (font (size 1 1) (thickness 0.15)))
     )
-    (fp_text user "${REFERENCE}" (at 0 -8.255 155) (layer "B.SilkS")
+    (fp_text user "${REFERENCE}" (at 0 -8.255 -25 unlocked) (layer "B.SilkS")
       (effects (font (size 1 1) (thickness 0.15)) (justify mirror))
     )
@@
     (property "Sheetname" "")
     (attr through_hole)
-    (fp_text reference "U1" (at 8.998955 -0.848008) (layer "B.SilkS")
-      (effects (font (size 1 1) (thickness 0.15)))
+    (fp_text reference "U1" (at 8.998955 -0.848008 unlocked) (layer "B.SilkS")
+      (effects (font (size 1 1) (thickness 0.15)) (justify mirror))
     )
     (fp_text value "YAAJ_WeAct_BlackPill_Part_Like" (at 20.32 24.765 90) (layer "F.Fab") hide
@@
     (property "Sheetname" "")
     (attr through_hole)
-    (fp_text reference "K31" (at 0 -8.255 170) (layer "F.SilkS")
+    (fp_text reference "K31" (at 0 -8.255 -10 unlocked) (layer "F.SilkS")
       (effects (font (size 1 1) (thickness 0.15)))
     )
@@
       (effects (font (size 1 1) (thickness 0.15)))
     )
-    (fp_text user "${REFERENCE}" (at 0 -8.255 170) (layer "B.SilkS")
+    (fp_text user "${REFERENCE}" (at 0 -8.255 -10 unlocked) (layer "B.SilkS")
       (effects (font (size 1 1) (thickness 0.15)) (justify mirror))
     )
@@
   (gr_line (start 154.3 46.270706) (end 140 46.270706) (layer "Edge.Cuts") (width 0.1))
   (gr_arc (start 141.8 122.600001) (mid 161.459797 123.564333) (end 180.129399 129.8) (layer "Edge.Cuts") (width 0.1))
+  (gr_text "U1" (at 38.1 20.32) (layer "B.SilkS")
+    (effects (font (size 1 1) (thickness 0.15)) (justify mirror))
+  )
   (gr_text "Cantor+" (at 187.15 84.4 90) (layer "B.SilkS")
     (effects (font (size 4 3) (thickness 0.4)) (justify mirror))
